File: build/keyboard/choc5x4_half.kicad_sch (KiCad schematic)
At the start: 40 parts, among them SW1 Choc V1/V2, SW10 Choc V1/V2, SW11 Choc V1/V2, SW12 Choc V1/V2, SW13 Choc V1/V2, SW14 Choc V1/V2, SW15 Choc V1/V2, SW16 Choc V1/V2, SW17 Choc V1/V2, SW18 Choc V1/V2, SW19 Choc V1/V2, SW2 Choc V1/V2, SW20 Choc V1/V2, SW3 Choc V1/V2, SW4 Choc V1/V2, SW5 Choc V1/V2, SW6 Choc V1/V2, SW7 Choc V1/V2, SW8 Choc V1/V2, SW9 Choc V1/V2

Commit message: update
Parts:
- added EH1: TPD1E05U06DYA, keyboard-design:sod523, symbol Interface:EH1
- added EH2: TPD1E05U06DYA, keyboard-design:sod523, symbol Interface:EH2
- added EH3: TPD1E05U06DYA, keyboard-design:sod523, symbol Interface:EH3
- added EH4: TPD1E05U06DYA, keyboard-design:sod523, symbol Interface:EH4
- added EH5: TPD1E05U06DYA, keyboard-design:sod523, symbol Interface:EH5
- added JH1: USB4115-03-C / GPIO ONLY, keyboard-design:usb4115, symbol Interface:JH1
- added RCH1: 1k contact isolation, keyboard-design:r0402, symbol Interface:RCH1
- added RCH10: 1k contact isolation, keyboard-design:r0402, symbol Interface:RCH10
- added RCH2: 1k contact isolation, keyboard-design:r0402, symbol Interface:RCH2
- added RCH3: 1k contact isolation, keyboard-design:r0402, symbol Interface:RCH3
- added RCH4: 1k contact isolation, keyboard-design:r0402, symbol Interface:RCH4
- added RCH5: 1k contact isolation, keyboard-design:r0402, symbol Interface:RCH5
- added RCH6: 1k contact isolation, keyboard-design:r0402, symbol Interface:RCH6
- added RCH7: 1k contact isolation, keyboard-design:r0402, symbol Interface:RCH7
- added RCH8: 1k contact isolation, keyboard-design:r0402, symbol Interface:RCH8
- added RCH9: 1k contact isolation, keyboard-design:r0402, symbol Interface:RCH9
- added RH1: 1k, keyboard-design:r0603, symbol Interface:RH1
- added RH2: 1k, keyboard-design:r0603, symbol Interface:RH2
- added RH3: 1k, keyboard-design:r0603, symbol Interface:RH3
- added RH4: 1k, keyboard-design:r0603, symbol Interface:RH4
- added RH5: 1k, keyboard-design:r0603, symbol Interface:RH5
Connections:
- net P0: now also RH1.2
- net P1: now also RH2.2
- net P2: now also RH3.2
- net P3: now also RH4.2
- net P4: now also RH5.2
- new net HC0: EH1.1, RCH1.2, RCH2.2, RH1.1
- new net HC1: EH2.1, RCH3.2, RCH4.2, RH2.1
- new net HC2: EH3.1, RCH5.2, RCH6.2, RH3.1
- new net HC3: EH4.1, RCH7.2, RCH8.2, RH4.1
- new net HC4: EH5.1, RCH10.2, RCH9.2, RH5.1
- new net H_A10: JH1.A10, RCH5.1
- new net H_A11: JH1.A11, RCH7.1
- new net H_A2: JH1.A2, RCH1.1
- new net H_A3: JH1.A3, RCH3.1
- new net H_A8: JH1.A8, RCH9.1
- new net H_B10: JH1.B10, RCH6.1
- new net H_B11: JH1.B11, RCH8.1
- new net H_B2: JH1.B2, RCH2.1
- new net H_B3: JH1.B3, RCH4.1
- new net H_B8: JH1.B8, RCH10.1
- new net SHIELD_H: EH1.2, EH2.2, EH3.2, EH4.2, EH5.2, JH1.S1, JH1.S2, JH1.S3, JH1.S4
- no-connect marks 0 -> 14
Other:
- note added: "USB-C interface below. VBUS / CC / USB2 / GND contacts NC. GPIO ONLY; electrical qualification pending."
- note removed: "No MCU, adapter, connector, power or inter-half wiring is selected in this matrix-only revision."

Commit message: WIP
Parts:
- D1, D10, D11, D12, D13, D14, D15, D16, D17, D18, D19, D2, D20, D3, D4, D5, D6, D7, D8, D9: value 1N4148W (candidate) -> 1N4148WT (candidate); footprint keyboard-design:diode_sod123 -> keyboard-design:diode_sod523
