File: build/keyboard/choc5x4_panel.kicad_pcb (KiCad board)
At the start: 2 copper layers, 98.2 x 99.5 mm, 106 parts, among them SW1 Kailh Choc V1 / V2, SW10 Kailh Choc V1 / V2, SW11 Kailh Choc V1 / V2, SW12 Kailh Choc V1 / V2, SW13 Kailh Choc V1 / V2, SW14 Kailh Choc V1 / V2, SW15 Kailh Choc V1 / V2, SW16 Kailh Choc V1 / V2, SW17 Kailh Choc V1 / V2, SW18 Kailh Choc V1 / V2, SW19 Kailh Choc V1 / V2, SW2 Kailh Choc V1 / V2, SW20 Kailh Choc V1 / V2, SW3 Kailh Choc V1 / V2, SW4 Kailh Choc V1 / V2, SW5 Kailh Choc V1 / V2, SW6 Kailh Choc V1 / V2, SW7 Kailh Choc V1 / V2, SW8 Kailh Choc V1 / V2, SW9 Kailh Choc V1 / V2, U1 XIAO SAMD21 / mount after dep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

Commit message: WIP
Parts:
- D1, D10, D11, D12, D13, D14, D15, D16, D17, D18, D19, D2, D20, D3, D4, D5, D6, D7, D8, D9: value 1N4148W -> 1N4148WT; footprint keyboard-design:diode_sod123 -> keyboard-design:diode_sod523
- JH1, JL, JR: moved to B.Cu
- moved EAL5 17.0 mm to (70.1, 140.0)
- moved EAR5 17.0 mm to (126.1, 140.0)
- moved EH5 15.6 mm to (52.0, 49.4)
- moved RCL2 15.4 mm to (72.5, 135.8)
- moved RCR2 15.4 mm to (123.7, 135.8)
- moved RCH1 14.8 mm to (66.6, 44.1)
- moved RCH3 14.7 mm to (66.6, 46.9)
- moved EAL4 14.2 mm to (70.1, 138.6)
- moved EAR4 14.2 mm to (126.1, 138.6)
- moved RCH2 12.9 mm to (66.6, 45.5)
- moved EH4 12.0 mm to (52.0, 48.1)
- moved EAL3 11.4 mm to (70.1, 137.2)
- moved EAR3 11.4 mm to (126.1, 137.2)
- moved RCL5 11.4 mm to (72.5, 140.0)
- moved RCR5 11.4 mm to (123.7, 140.0)
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